Commit message: add simplified utv3 mesh

File: kuka_omnimove_e575_support/urdf/omnimove.xacro (robot description, xacro)
@@ -7,21 +7,20 @@
           <origin xyz="0 0 0" rpy="0 0 0" />
           <geometry>
-            <mesh filename="package://kuka_omnimove_e575_support/meshes/omnimove_simplified.dae" />
+            <mesh filename="package://kuka_omnimove_e575_support/meshes/quantec_simplified.dae" />
           </geometry>
+          <!--<xacro:material_kuka_pedestal /> -->
         </visual>
         <collision>
           <origin xyz="0 0 0" rpy="0 0 0" />
           <geometry>
-            <mesh filename="package://kuka_omnimove_e575_support/meshes/omnimove_simplified.stl" />
+            <mesh filename="package://kuka_omnimove_e575_support/meshes/quantec_simplified.stl" />
           </geometry>
         </collision>
       </link>
   </xacro:macro>
-   <xacro:macro name="omnimove_ros2_control" params="name">
-	    <ros2_control name="omnimove" type="system">
+  <xacro:macro name="omnimove_ros2_control" params="name">
+      <ros2_control name="omnimove" type="system">
             <hardware>
                 <plugin>omnimove::OmnimoveExternalControl</plugin>
-                <param name ="host">127.0.0.1</param>
-                <param name="port">24000</param>
             </hardware>
             <joint name="move_x">
@@ -45,5 +44,5 @@
                 <state_interface name="velocity"/>
             </joint>
-	   </ros2_control>
+      </ros2_control>
   </xacro:macro>
 </robot>

File: kuka_omnimove_e575_support/urdf/omnimove_with_arm.xacro (robot description, xacro)
@@ -1,11 +1,12 @@
 <?xml version="1.0" ?>
 <robot name="kuka_kr6r700sixx" xmlns:xacro="http://wiki.ros.org/xacro">
-        <xacro:include filename="$(find kuka_quantec_support)/urdf/kr210_r2700-2.urdf.xacro"/>
+  <xacro:include filename="$(find kuka_quantec_support)/urdf/kr210_r2700-2.urdf.xacro"/>
   <xacro:include filename="$(find kuka_omnimove_e575_support)/urdf/omnimove.xacro"/>
   <xacro:omnimove prefix="omnimove_"/>
-       <!--  <xacro:omnimove_ros2_control name="omnimove"/> -->
+  <xacro:omnimove_ros2_control name="omnimove"/>
   <joint name="omnibase" type="fixed">
     <parent link="omnimove_base"/>
     <child link="base_link"/>
+    <origin xyz="0.89567 0.00247 0.48018"/>
   </joint>
 </robot>
